Commit message: 已完成mid360无人车仿真环境的搭建

File: src/ground_shark_description/urdf/Ground-Shark_description_fixed.gazebo.xacro (robot description, xacro)
@@ -125,5 +125,5 @@
         <bodyName>imu_link</bodyName>
         <updateRateHZ>200.0</updateRateHZ>
-        <gaussianNoise>0.0</gaussianNoise>
+        <gaussianNoise>0.00329</gaussianNoise>
         <xyzOffset>0 0 0</xyzOffset>
         <rpyOffset>0 0 0</rpyOffset>

File: src/ground_shark_mid360/urdf/ground_shark_mid360_fixed.urdf (robot description, URDF)
Before this commit: robot ground_shark_mid360, 16 links, 15 joints
Links:
- added link camera_link, mass 0.073513; collision box size=0.1 0.05 0.05; visual box size=0.05 0.1 0.05
- link imu_link: mass 0 -> 0.02; geometry visual mesh filename=package://ground_shark_mid360/meshes/imu_link.STL
- link lidar_link: geometry visual mesh filename=package://ground_shark_mid360/meshes/lidar_link.STL
Joints:
- added joint camera_joint: type fixed, parent base_link, child camera_link, origin xyz=0.12 0 0.04 rpy=0 0 0, axis 0 0 0

File: src/ground_shark_mid360/urdf/mid360_gazebo.xacro (robot description, xacro)
@@ -1,9 +1,10 @@
 <?xml version="1.0" encoding="utf-8"?>
 <!-- Livox Mid360 仿真插件（可复用于任何机器人） -->
-<!-- 从官方仿真驱动库部分截取而来，保留了传感器部分，删除了视觉碰撞模型部分和搭载底盘部分 -->
+<!-- 从官方仿真驱动库部分截取而来，保留了传感器部分，增加了IMU传感器，删除了视觉碰撞模型部分和搭载底盘部分 -->
 <robot xmlns:xacro="http://ros.org/wiki/xacro">
     <xacro:property name="M_PI" value="3.14159"/>
     <xacro:property name="laser_min_range" value="0.1"/>
-    <xacro:property name="laser_max_range" value="200.0"/>
+    <!-- <xacro:property name="laser_max_range" value="200.0"/> -->
+    <xacro:property name="laser_max_range" value="30.0"/>
     <xacro:property name="ros_topic" value="scan"/>
     <xacro:property name="samples" value="24000"/>
@@ -11,51 +12,72 @@
     <xacro:macro name="null_inertial">
         <inertial>
-        <mass value="0.1"/>
-        <inertia ixx="0.01" ixy="0" ixz="0"
-            iyy="0.01" iyz="0"
-            izz="0.01"/>
+            <mass value="0.1"/>
+            <inertia ixx="0.01" ixy="0" ixz="0" iyy="0.01" iyz="0" izz="0.01"/>
         </inertial>
     </xacro:macro>
-    <xacro:macro name="Livox_Mid_gazebo_sensor" params="visualize:=True update_rate:=10 resolution:=0.002 noise_mean:=0.0 noise_stddev:=0.01 name:=livox ros_topic:=${ros_topic}">
+    <xacro:macro name="Livox_Mid_gazebo_sensor" params="visualize:=true update_rate:=10 resolution:=0.002 noise_mean:=0.0 noise_stddev:=0.01 name:=livox ros_topic:=${ros_topic}">
         <gazebo reference="${name}">
-        <sensor type="ray" name="laser_${name}">
-            <pose>0 0 0 0 0 0</pose>
-            <visualize>${visualize}</visualize>
-            <update_rate>${update_rate}</update_rate>
-            <!-- This ray plgin is only for visualization. -->
-            <plugin name="gazebo_ros_laser_controller" filename="liblivox_laser_simulation.so">
-                <ray>
-                <scan>
-                    <horizontal>
-                        <samples>100</samples>
-                        <resolution>1</resolution>
-                        <min_angle>0</min_angle>
+            <sensor type="ray" name="laser_${name}">
+                <pose>0 0 0 0 0 0</pose>
+                <visualize>${visualize}</visualize>
+                <update_rate>${update_rate}</update_rate>
+                <!-- This ray plgin is only for visualization. -->
+                <plugin name="gazebo_ros_laser_controller" filename="liblivox_laser_simulation.so">
+                    <ray>
+                        <scan>
+                            <horizontal>
+                                <samples>100</samples>
+                                <resolution>1</resolution>
+                                <min_angle>${0}</min_angle>
                                 <max_angle>${(2)*M_PI}</max_angle>
-                    </horizontal>
-                    <vertical>
-                        <samples>360</samples>
-                        <resolution>1</resolution>
-                        <min_angle>${(-3.22)/180*M_PI}</min_angle>
-                            <max_angle>${(56.22)/180*M_PI}</max_angle>
-                    </vertical>
-                </scan>
-                <range>
-                    <min>0.1</min>
-                    <max>30</max>
-                    <resolution>0.02</resolution>
-                </range>
-                <noise>
-                    <type>gaussian</type>
-                    <mean>0.0</mean>
-                    <stddev>0.0</stddev>
-                </noise>
-                </ray>
-            <visualize>${visualize}</visualize>
-            <samples>${samples}</samples>
-            <downsample>${downsample}</downsample>
-            <csv_file_name>package://livox_laser_simulation/scan_mode/mid360.csv</csv_file_name>
-            <ros_topic>${ros_topic}</ros_topic>
-            </plugin>
-        </sensor>
+                            </horizontal>
+                            <vertical>
+                                <samples>360</samples>
+                                <resolution>1</resolution>
+                                <min_angle>${(-3.22)/180*M_PI}</min_angle>
+                                <max_angle>${(56.22)/180*M_PI}</max_angle>
+                            </vertical>
+                        </scan>
+                        <range>
+                            <min>${laser_min_range}</min>
+                            <max>${laser_max_range}</max>
+                            <resolution>${resolution}</resolution>
+                        </range>
+                        <noise>
+                            <type>gaussian</type>
+                            <mean>${noise_mean}</mean>
+                            <stddev>${noise_stddev}</stddev>
+                        </noise>
+                    </ray>
+                    <scan_mode>Mid360</scan_mode>
+                    <visualize>${visualize}</visualize>
+                    <samples>${samples}</samples>
+                    <downsample>${downsample}</downsample>
+                    <csv_file_name>package://livox_laser_simulation/scan_mode/mid360.csv</csv_file_name>
+                    <ros_topic>${ros_topic}</ros_topic>
+                </plugin>
+            </sensor>
+        </gazebo>
+    </xacro:macro>
+    <xacro:macro name="Livox_Mid_gazebo_imu" params="visualize:=true update_rate:=200 gaussianNoise:=0.00329 name:=livox ros_topic:=/livox/imu">
+        <!-- 在 IMU_Link 上加载IMU测量插件检测运动 -->
+        <gazebo reference="${name}">
+            <gravity>true</gravity>
+            <sensor name="${name}_imu" type="imu">
+                <always_on>true</always_on>
+                <update_rate>${update_rate}</update_rate>
+                <visualize>${visualize}</visualize>
+                <plugin name="imu_plugin" filename="libgazebo_ros_imu_sensor.so">
+                    <topicName>${ros_topic}</topicName>
+                    <bodyName>${name}</bodyName>
+                    <updateRateHZ>${update_rate}</updateRateHZ>
+                    <gaussianNoise>${gaussianNoise}</gaussianNoise>
+                    <xyzOffset>0 0 0</xyzOffset>
+                    <rpyOffset>0 0 0</rpyOffset>
+                    <frameName>${name}</frameName>
+                    <initialOrientationAsReference>false</initialOrientationAsReference>
+                </plugin>
+                <pose>0 0 0 0 0 0</pose>
+            </sensor>
         </gazebo>
     </xacro:macro>

File: src/ground_shark_mid360/urdf/my_ground_robot_mid360.xacro (robot description, xacro)
@@ -2,17 +2,21 @@
 <!-- 地面麦轮小车 + Mid360 -->
 <!-- 关节连接基于base_link——lidar_link——imu_link -->
-<robot
-    name="ground_shark_mid360" xmlns:xacro="http://ros.org/wiki/xacro">
-    <!-- 1. 引入带有雷达模型的地面麦轮小车 -->
-    <xacro:include
-        filename="$(find ground_shark_mid360)/urdf/ground_shark_mid360_fixed.urdf" />
-    <!-- 2. 引入雷达仿真宏并调用→ 自动生成 Gazebo 仿真传感器（关键！） -->
+<robot name="ground_shark_mid360"
+    xmlns:xacro="http://ros.org/wiki/xacro">
+    <!-- 引入带有雷达模型的地面麦轮小车 -->
+    <xacro:include filename="$(find ground_shark_mid360)/urdf/ground_shark_mid360_fixed.urdf" />
+    <!-- 设置摩擦系数 -->
+    <xacro:include filename="$(find ground_shark_mid360)/urdf/basic_gazebo_plugins.xacro" />
+    <xacro:default_link link_name="wheel_fl_link" />
+    <xacro:default_link link_name="wheel_fr_link" />
+    <xacro:default_link link_name="wheel_bl_link" />
+    <xacro:default_link link_name="wheel_br_link" />
+    <xacro:default_link link_name="base_link" />
+    <!-- 引入万向控制插件控制车体 -->
+    <xacro:gazebo_ros_planner_move cmd_topic="cmd_vel" frame="base_footprint"  />
+    <!-- 引入雷达和IMU仿真宏并调用→ 自动生成 Gazebo 仿真传感器（关键！） -->
     <xacro:include filename="$(find ground_shark_mid360)/urdf/mid360_gazebo.xacro" />
-    <xacro:Livox_Mid_gazebo_sensor
-        name="lidar_link"
-        visualize="true"
-        update_rate="10"
-        ros_topic="/livox/lidar"
-    />
+    <xacro:Livox_Mid_gazebo_sensor name="lidar_link" visualize="true" update_rate="10" ros_topic="/livox/lidar" />
+    <xacro:Livox_Mid_gazebo_imu name="imu_link" visualize="true" update_rate="200" ros_topic="/livox/imu" gaussianNoise="0.0" />
     <!-- 设置属性变好看一点 -->
     <gazebo reference="wheel_fl_link">
@@ -29,8 +33,14 @@
     </gazebo>
     <gazebo reference="imu_link">
-        <material>Gazebo/White</material>
+        <material>Gazebo/Green</material>
     </gazebo>
     <gazebo reference="lidar_link">
         <material>Gazebo/Blue</material>
     </gazebo>
+    <gazebo reference="camera_link">
+        <material>Gazebo/Red</material>
+    </gazebo>
+    <!-- 引入一个相机仿真宏 -->
+    <xacro:include filename="$(find ground_shark_mid360)/urdf/camera_gazebo.xacro" />
+    <xacro:sensor_camera name="my_camera" update_rate="30.0" image_topic="image_raw" frame="camera_link" />
 </robot>
